File: KiCad/PCB/Sigilv1/Sigilv1.kicad_sch (KiCad schematic)
At the start: 11 parts, among them SW1 PASS, SW2 ACTION, SW3 ACTION / WIN, SW4 PAIR, U1 ESP32-WROOM-32E

Commit message: KiCad Schematic Update
Parts:
- removed SW3: ACTION / WIN, symbol Switch:SW_Push
- removed U1: ESP32-WROOM-32E, RF_Module:ESP32-WROOM-32E, symbol RF_Module:ESP32-WROOM-32E
- added J2: EPD LOGICAL ONLY, symbol Sigil:EPD_Logical_Interface
- added J3: BUZZER LOGICAL ONLY, symbol Sigil:Buzzer_Logical_Interface
- added U1: REMOVABLE ESP32 DEVKIT / 2 x 19, symbol Sigil:ESP32_DevKit_38_RearReference
- D1: value RED STATUS -> RED
- D2: value GREEN STATUS -> GREEN
- D3: value BLUE STATUS -> BLUE
- SW1: value PASS -> BTN_PASS
- SW2: value ACTION -> BTN_ACTION
Connections:
- net +3V3: now also J2.VCC, U1.J19 (3V3)
- net BTN_ACTION: now also U1.J11 (GPIO25 / BTN_ACTION)
- net BTN_PASS: now also U1.J10 (GPIO26 / BTN_PASS)
- net BUZZER: now also J3.SIG, U1.J12 (GPIO33 / BUZZER)
- net EPD_BUSY: now also J2.BUSY, U1.A14 (GPIO21 / EPD_BUSY)
- net EPD_CS: now also J2.CS, U1.A9 (GPIO17 / EPD_CS)
- net EPD_DC: now also J2.DC, U1.A8 (GPIO16 / EPD_DC)
- net EPD_MOSI: now also J2.DIN, U1.A18 (GPIO23 / EPD_MOSI)
- net EPD_RST: now also J2.RST, U1.A17 (GPIO22 / EPD_RST)
- net EPD_SCLK: now also J2.CLK, U1.A11 (GPIO18 / EPD_SCLK)
- net GND: now also D1.1 (K), D2.1 (K), D3.1 (K), J2.GND, J3.GND, U1.A13 (GND), U1.A19 (GND), U1.J6 (GND); no longer D1.2 (A), D2.2 (A), D3.2 (A)
- net LED_BLUE: now also U1.J9 (GPIO27 / LED_BLUE)
- net LED_GREEN: now also U1.J8 (GPIO14 / LED_GREEN)
- net LED_RED: now also U1.J5 (GPIO13 / LED_RED)
- net at R3.2: now also D3.2 (A)
- net at R2.2: now also D2.2 (A)
- net at R1.2: now also D1.2 (A)
- net BTN_PAIR renamed PAIR
- net PAIR: now also U1.A12 (GPIO19 / PAIR)
- no-connect marks 0 -> 21
Other:
- note added: "330R retained from existing schematic; LED part/current verification remains open."
- note added: "BACK / REAR PHOTO VIEW J1 top-left; A1 top-right Socket IDs are immutable; this is NOT a footprint view."
- note added: "CONTROLS - INPUT_PULLUP"
- note added: "J3 is an unresolved load interface. Confirm transducer/driver, current and protection. No direct-drive suitability is assumed."
- note added: "PAIR: A12 / GPIO19 to A13 / GND Released HIGH; pressed LOW. No carrier BOOT or reset circuitry."
- note added: "SCHEMATIC REVIEW / RELEASE HOLDS 1. U1 uses A1-A19 / J1-J19 from SigilBackMarked.png (BACK view); never exchange row identities. 2. No DevKit footprint assigned: measure pitch, row spacing, outline, USB-C overhang, holes, socket height and keepouts. 3. Future footprint: two 1x19 female sockets, unmistakable A1/J1 marks; verify insertion from carrier component side. 4. Keep USB-C, BOOT and EN/rese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"
- note added: "STATUS LEDS - active HIGH"
- note added: "USB-powered DevKit; J1 / 5V unused on carrier. J19 supplies +3V3. All three GND sockets connected. Onboard USB-UART, regulator, BOOT and EN retained."
- note added: "Write-only display; no MISO connection. J2 names are logical signals, NOT physical pin numbers. Confirm module, VCC rating and connector order."
- note removed: "CONTROLS (active-low, firmware INPUT_PULLUP)"
- note removed: "E-PAPER INTERFACE"
- note removed: "EPD connector/header symbol to be finalized after display module is confirmed."
- note removed: "GPIO19 = PAIR (future) | GPIO4 = ACTION/WIN auxiliary (future)"
- note removed: "NOTE: U1 is the bare ESP32-WROOM-32E module; +3V3/GND are explicitly assigned."
- note removed: "STATUS LEDS - 330R current-limit resistors"
- note removed: "TURNHUB SIGIL REV A - FUNCTIONAL PROTOTYPE"
- title: (none) -> Sigil Rev A - removable DevKit carrier
