File: KiCad/PCB/Sigilv1/Sigilv1.kicad_sch (KiCad schematic)
At the start: 12 parts, among them J2 EPD LOGICAL ONLY, J3 BUZZER LOGICAL ONLY, SW1 BTN_PASS, SW2 BTN_ACTION, SW4 PAIR, U1 REMOVABLE ESP32 DEVKIT / 2 x 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

Commit message: Add the Pause/Win button to the Sigil Rev A schematic
Firmware (PAUSE_WIN_BUTTON = 32) and HARDWARE_REFERENCE.md put the
Pause/Win button on GPIO32 / socket J13. The schematic had only a
hand-added BTN_PAUSE label with no switch, so the net was one-ended and
the embedded U1 symbol no longer matched Sigil.kicad_sym.

build_schematic.py now draws SW5 from BTN_PAUSE to GND and names the
J13 pin; verify_schematic.py checks the new mapping and switch. The
script also emits deterministic pin UUIDs and re-saves through
kicad-cli when available, so its output matches KiCad's own format.
KiCad 10.0.6 ERC: 0 errors, 0 warnings.

Co-Authored-By: Claude Opus 5.5 <noreply@anthropic.com>
Claude-Session: https://claude.ai/code/session_01RYQ71iURGsU5zU9bGT83PG
Parts:
- added SW5: BTN_PAUSE, symbol Switch:SW_Push
Connections:
- net BTN_PAUSE: now also SW5.1
- net GND: now also SW5.2
- no-connect marks 21 -> 20
Other:
- note added: "PAIR: A12 / GPIO19 to A13 / GND PAUSE/WIN: J13 / GPIO32 to GND (SW3 retired) All released HIGH; pressed LOW. No carrier BOOT or reset circuitry."
- note removed: "PAIR: A12 / GPIO19 to A13 / GND Released HIGH; pressed LOW. No carrier BOOT or reset circuitry."
