File: KiCad/PCB/Sigilv1/Sigilv1.kicad_sch (KiCad schematic)
At the start: 13 parts, among them J2 EPD LOGICAL ONLY, J3 BUZZER LOGICAL ONLY, SW1 BTN_PASS, SW2 BTN_ACTION, SW4 PAIR, SW5 BTN_PAUSE, U1 REMOVABLE ESP32 DEVKIT / 2 x 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

Commit message: New Atlas!!!
Connections:
- net +3V3: now also U1.A11 (3V3); no longer U1.J19 (3V3)
- net BTN_ACTION: now also U1.A19 (GPIO25_/_BTN_ACTION); no longer U1.J11 (GPIO25_/_BTN_ACTION)
- net BTN_PASS: now also U1.A20 (GPIO26_/_BTN_PASS); no longer U1.J10 (GPIO26_/_BTN_PASS)
- net BTN_PAUSE: now also U1.A17 (GPIO32_/_BTN_PAUSE); no longer U1.J13 (GPIO32_/_BTN_PAUSE)
- net BUZZER: now also U1.A18 (GPIO33_/_BUZZER); no longer U1.J12 (GPIO33_/_BUZZER)
- net EPD_BUSY: now also U1.J16 (GPIO21_/_EPD_BUSY); no longer U1.A14 (GPIO21_/_EPD_BUSY)
- net EPD_CS: now also U1.J21 (GPIO17_/_EPD_CS); no longer U1.A9 (GPIO17_/_EPD_CS)
- net EPD_DC: now also U1.J22 (GPIO16_/_EPD_DC); no longer U1.A8 (GPIO16_/_EPD_DC)
- net EPD_MOSI: now also U1.J12 (GPIO23_/_EPD_MOSI); no longer U1.A18 (GPIO23_/_EPD_MOSI)
- net EPD_RST: now also U1.J13 (GPIO22_/_EPD_RST); no longer U1.A17 (GPIO22_/_EPD_RST)
- net EPD_SCLK: now also U1.J19 (GPIO18_/_EPD_SCLK); no longer U1.A11 (GPIO18_/_EPD_SCLK)
- net GND: now also U1.A24 (GND), U1.J11 (GND), U1.J17 (GND); no longer U1.A13 (GND), U1.A19 (GND), U1.J6 (GND)
- net LED_BLUE: now also U1.A21 (GPIO27_/_LED_BLUE); no longer U1.J9 (GPIO27_/_LED_BLUE)
- net LED_GREEN: now also U1.A22 (GPIO14_/_LED_GREEN); no longer U1.J8 (GPIO14_/_LED_GREEN)
- net LED_RED: now also U1.A25 (GPIO13_/_LED_RED); no longer U1.J5 (GPIO13_/_LED_RED)
- net PAIR: now also U1.J18 (GPIO19_/_PAIR); no longer U1.A12 (GPIO19_/_PAIR)
Other:
- note added: "BACK / REAR PHOTO VIEW A29 top-left; J29 top-right (breadboard rotated 180 degrees) This is NOT a footprint view."
- note added: "PAIR: J18 / GPIO19 to J17 / GND PAUSE/WIN: A17 / GPIO32 to GND (SW3 retired) All released HIGH; pressed LOW. No carrier BOOT or reset circuitry."
- note added: "SCHEMATIC REVIEW / RELEASE HOLDS 1. U1 uses A11-A29 / J11-J29 after the 180-degree breadboard rotation (old An = J(30-n), old Jn = A(30-n)). SigilBackMarked.png (BACK view) still shows the pre-rotation A1-A19 / J1-J19 labels. 2. No DevKit footprint assigned: measure pitch, row spacing, outline, USB-C overhang, holes, socket height and keepouts. 3. Future footprint: two 1x19 female sockets, unmist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"
- note added: "USB-powered DevKit; A29 / 5V unused on carrier. A11 supplies +3V3. All three GND sockets connected. Onboard USB-UART, regulator, BOOT and EN retained."
- note removed: "BACK / REAR PHOTO VIEW J1 top-left; A1 top-right Socket IDs are immutable; this is NOT a footprint view."
- note removed: "PAIR: A12 / GPIO19 to A13 / GND PAUSE/WIN: J13 / GPIO32 to GND (SW3 retired) All released HIGH; pressed LOW. No carrier BOOT or reset circuitry."
- note removed: "SCHEMATIC REVIEW / RELEASE HOLDS 1. U1 uses A1-A19 / J1-J19 from SigilBackMarked.png (BACK view); never exchange row identities. 2. No DevKit footprint assigned: measure pitch, row spacing, outline, USB-C overhang, holes, socket height and keepouts. 3. Future footprint: two 1x19 female sockets, unmistakable A1/J1 marks; verify insertion from carrier component side. 4. Keep USB-C, BOOT and EN/rese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"
- note removed: "USB-powered DevKit; J1 / 5V unused on carrier. J19 supplies +3V3. All three GND sockets connected. Onboard USB-UART, regulator, BOOT and EN retained."
Changed lines of the file:
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@@
-		)
-	)
-	(text "BACK / REAR PHOTO VIEW\nJ1 top-left; A1 top-right\nSocket IDs are immutable; this is NOT a footprint view."
-		(exclude_from_sim no)
-		(at 28 21 0)
-		(effects
-			(font
-				(size 1.5 1.5)
-			)
-			(justify left top)
 		)
 	)
@@
 		)
 	)
-	(text "USB-powered DevKit; J1 / 5V unused on carrier.\nJ19 supplies +3V3. All three GND sockets connected.\nOnboard USB-UART, regulator, BOOT and EN retained."
+	(text "PAIR: J18 / GPIO19 to J17 / GND\nPAUSE/WIN: A17 / GPIO32 to GND (SW3 retired)\nAll released HIGH; pressed LOW.\nNo carrier BOOT or reset circuitry."
+		(exclude_from_sim no)
+		(at 175 130 0)
+		(effects
+			(font
+				(size 1.27 1.27)
+			)
+			(justify left top)
+		)
+	)
+	(text "USB-powered DevKit; A29 / 5V unused on carrier.\nA11 supplies +3V3. All three GND sockets connected.\nOnboard USB-UART, regulator, BOOT and EN retained."
 		(exclude_from_sim no)
 		(at 28 157 0)
@@
 		)
 	)
-	(text "PAIR: A12 / GPIO19 to A13 / GND\nPAUSE/WIN: J13 / GPIO32 to GND (SW3 retired)\nAll released HIGH; pressed LOW.\nNo carrier BOOT or reset circuitry."
-		(exclude_from_sim no)
-		(at 175 130 0)
-		(effects
-			(font
-				(size 1.27 1.27)
-			)
-			(justify left top)
-		)
-	)
-	(text "SCHEMATIC REVIEW / RELEASE HOLDS\n1. U1 uses A1-A19 / J1-J19 from SigilBackMarked.png (BACK view); never exchange row identities.\n2. No DevKit footprint assigned: measure pitch, row spacing, outline, USB-C overhang, holes, socket height and keepouts.\n3. Future footprint: two 1x19 female sockets, unmistakable A1/J1 marks; verify insertion from carrier component side.\n4. Keep USB-C, BOOT and EN/reset accessible; preserve antenna/component clearances after measurement.\n5. Display connector and buzzer circuit are unresolved logical interfaces, excluded from PCB and BOM.\n6. Old GPIO4 auxiliary and GPIO32 display-detect removed; GPIO32 / J13 is now the Pause/Win button (SW5).\n7. Rev A is an electrical draft, NOT fabrication-ready. Power through DevKit USB; no second supply designed."
+	(text "SCHEMATIC REVIEW / RELEASE HOLDS\n1. U1 uses A11-A29 / J11-J29 after the 180-degree breadboard rotation (old An = J(30-n), old Jn = A(30-n)).\n   SigilBackMarked.png (BACK view) still shows the pre-rotation A1-A19 / J1-J19 labels.\n2. No DevKit footprint assigned: measure pitch, row spacing, outline, USB-C overhang, holes, socket height and keepouts.\n3. Future footprint: two 1x19 female sockets, unmistakable A29/J29 marks; verify insertion from carrier component side.\n4. Keep USB-C, BOOT and EN/reset accessible; preserve antenna/component clearances after measurement.\n5. Display connector and buzzer circuit are unresolved logical interfaces, excluded from PCB and BOM.\n6. Old GPIO4 auxiliary and GPIO32 display-detect removed; GPIO32 / A17 is now the Pause/Win button (SW5).\n7. Rev A is an electrical draft, NOT fabrication-ready. Power through DevKit USB; no second supply designed."
 		(exclude_from_sim no)
 		(at 28 211 0)
@@
 		(exclude_from_sim no)
 		(at 175 40 0)
+		(effects
+			(font
+				(size 1.5 1.5)
+			)
+			(justify left top)
+		)
+	)
+	(text "BACK / REAR PHOTO VIEW\nA29 top-left; J29 top-right (breadboard rotated 180 degrees)\nThis is NOT a footprint view."
+		(exclude_from_sim no)
+		(at 28 21 0)
 		(effects
 			(font
@@
 			)
 		)
-		(pin "J1"
-		)
-		(pin "J2"
-		)
-		(pin "J3"
-		)
-		(pin "J4"
-		)
-		(pin "J5"
-		)
-		(pin "J6"
-		)
-		(pin "J7"
-		)
-		(pin "J8"
-		)
-		(pin "J9"
-		)
-		(pin "J10"
+		(pin "A29"
+		)
+		(pin "A28"
+		)
+		(pin "A27"
+		)
+		(pin "A26"
+		)
+		(pin "A25"
+		)
+		(pin "A24"
+		)
+		(pin "A23"
+		)
+		(pin "A22"
+		)
+		(pin "A21"
+		)
+		(pin "A20"
+		)
+		(pin "A19"
+		)
+		(pin "A18"
+		)
+		(pin "A17"
+		)
+		(pin "A16"
+		)
+		(pin "A15"
+		)
+		(pin "A14"
+		)
+		(pin "A13"
+		)
+		(pin "A12"
+		)
+		(pin "A11"
+		)
+		(pin "J29"
+		)
+		(pin "J28"
+		)
+		(pin "J27"
+		)
+		(pin "J26"
+		)
+		(pin "J25"
+		)
+		(pin "J24"
+		)
+		(pin "J23"
+		)
+		(pin "J22"
+		)
+		(pin "J21"
+		)
+		(pin "J20"
+		)
+		(pin "J19"
+		)
+		(pin "J18"
+		)
+		(pin "J17"
+		)
+		(pin "J16"
+		)
+		(pin "J15"
+		)
+		(pin "J14"
+		)
+		(pin "J13"
+		)
+		(pin "J12"
 		)
 		(pin "J11"
 		)
-		(pin "J12"
-		)
-		(pin "J13"
-		)
-		(pin "J14"
-		)
-		(pin "J15"
-		)
-		(pin "J16"
-		)
-		(pin "J17"
-		)
-		(pin "J18"
-		)
-		(pin "J19"
-		)
-		(pin "A1"
-		)
-		(pin "A2"
-		)
-		(pin "A3"
-		)
-		(pin "A4"
-		)
-		(pin "A5"
-		)
-		(pin "A6"
-		)
-		(pin "A7"
-		)
-		(pin "A8"
-		)
-		(pin "A9"
-		)
-		(pin "A10"
-		)
-		(pin "A11"
-		)
-		(pin "A12"
-		)
-		(pin "A13"
-		)
-		(pin "A14"
-		)
-		(pin "A15"
-		)
-		(pin "A16"
-		)
-		(pin "A17"
-		)
-		(pin "A18"
-		)
-		(pin "A19"
-		)
 		(instances
