File: KiCad/PCB/Sigilv1/Sigil_EInk.kicad_pcb (KiCad board)
At the start: 2 copper layers, 9 parts, among them J2 INLAND E-PAPER HEADER (8-PIN), J3 BUZZER 2-PIN HEADER, J4 ANALOG JOYSTICK HEADER (5-PIN), J5 STATUS RING CABLE (JST-XH 3), U1 REMOVABLE ESP32 DEVKIT / 2 x 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, U2 74AHCT1G125

Commit message: PCB Work
Parts:
- added C4: 100nF, Capacitor_THT:C_Disc_D5.0mm_W2.5mm_P5.00mm, F.Cu at (109.5, 165.5)
- added H1: M3, MountingHole:MountingHole_3.2mm_M3, F.Cu at (104.0, 104.0)
- added H2: M3, MountingHole:MountingHole_3.2mm_M3, F.Cu at (142.0, 104.0)
- added H3: M3, MountingHole:MountingHole_3.2mm_M3, F.Cu at (104.0, 172.0)
- added H4: M3, MountingHole:MountingHole_3.2mm_M3, F.Cu at (142.0, 172.0)
- added J6: FRONT LIGHT CABLE (JST-XH 3), Connector_JST:JST_XH_B3B-XH-A_1x03_P2.50mm_Vertical, F.Cu at (120.5, 170.5)
- added R2: 330R, Resistor_THT:R_Axial_DIN0207_L6.3mm_D2.5mm_P7.62mm_Horizontal, F.Cu at (122.2, 160.0)
- added U3: 74AHCT1G125, Package_TO_SOT_SMD:SOT-23-5, F.Cu at (112.0, 160.1)
- J2: footprint Connector_PinSocket_2.54mm:PinSocket_1x08_P2.54mm_Vertical -> Connector_JST:JST_XH_B8B-XH-A_1x08_P2.50mm_Vertical
- J4: footprint Connector_PinSocket_2.54mm:PinSocket_1x05_P2.54mm_Vertical -> Connector_JST:JST_XH_B5B-XH-A_1x05_P2.50mm_Vertical
- moved J3 153.7 mm to (132.0, 166.7)
- moved R1 128.0 mm to (141.8, 142.8), turned to 90 degrees
- moved J2 123.6 mm to (104.3, 144.8), turned to 90 degrees
- moved U2 115.5 mm to (141.8, 122.6)
- moved C2 112.2 mm to (104.8, 154.0), turned to 90 degrees
- moved C3 97.8 mm to (141.8, 132.0), turned to 90 degrees
- moved J4 97.2 mm to (141.3, 159.0), turned to 90 degrees
- moved U1 83.5 mm to (111.6, 103.4)
- moved J5 68.8 mm to (141.3, 116.5), turned to 90 degrees
Connections:
- U1 pad J5: unconnected-(U1-GPIO13-PadJ5) -> /FRONT_DIN
Routing:
- added copper zone on B.Cu, net /GND
Other:
- board outline added: 46 x 76 mm
