File: KiCad/PCB/Sigilv1/Sigil_EInk.kicad_sch (KiCad schematic)
At the start: 9 parts, among them J2 INLAND E-PAPER HEADER (8-PIN), J3 BUZZER 2-PIN HEADER, J4 ANALOG JOYSTICK HEADER (5-PIN), J5 STATUS RING CABLE (JST-XH 3), U1 REMOVABLE ESP32 DEVKIT / 2 x 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, U2 74AHCT1G125

Commit message: PCB Work
Parts:
- added C4: 100nF, Capacitor_THT:C_Disc_D5.0mm_W2.5mm_P5.00mm, symbol Sigil:Capacitor
- added J6: FRONT LIGHT CABLE (JST-XH 3), Connector_JST:JST_XH_B3B-XH-A_1x03_P2.50mm_Vertical, symbol Sigil:Front_Cable_JST_XH_3
- added R2: 330R, Resistor_THT:R_Axial_DIN0207_L6.3mm_D2.5mm_P7.62mm_Horizontal, symbol Sigil:Resistor_Series
- added U3: 74AHCT1G125, Package_TO_SOT_SMD:SOT-23-5, symbol Sigil:74AHCT1G125
- J2: footprint Connector_PinSocket_2.54mm:PinSocket_1x08_P2.54mm_Vertical -> Connector_JST:JST_XH_B8B-XH-A_1x08_P2.50mm_Vertical
- J4: footprint Connector_PinSocket_2.54mm:PinSocket_1x05_P2.54mm_Vertical -> Connector_JST:JST_XH_B5B-XH-A_1x05_P2.50mm_Vertical
Connections:
- net +5V: now also C4.1, J6.1 (+5V), U3.5 (VCC)
- net GND: now also C4.2, J6.3 (GND), U3.1 (OE#), U3.3 (GND)
- net FRONT_DIN: now reaches U1.J5 (GPIO13)
- net FRONT_DIN: now also U3.2 (A)
- new net FRONT_DIN_5V: R2.1, U3.4 (Y)
- new net FRONT_DIN_R: J6.2 (DIN), R2.2
- no-connect marks 22 -> 21
Other:
- note added: "FRONT LIGHT (SPARE OUTPUT)"
- note added: "J6: spare front light output, e.g. 6-8 SK6812 RGBW pixels on the case front lip facing the seated player. Own data line: GPIO13 -> U3 (74AHCT1G125, C4) -> R2 (330 ohm) -> DIN; pinout as J5. Shares USB 5V with the ring: firmware must cap both (7 + 8 pixels at 48/255 is about 225 mA). Fitted; unused until a strip is added."
- note added: "SCHEMATIC REVIEW / RELEASE HOLDS 1. U1 uses A1-A19 / J1-J19 from SigilBackMarked.png (BACK view); never exchange row identities. 2. U1 footprint (Sigil.pretty): 2.54 mm pitch, rows 22.86 mm (0.9 in) apart from the breadboard fit (Inland publishes 25.4 mm), 53.9 x 27.5 mm outline (length from the breadboard fit). Caliper-check and test-fit before ordering. 3. Future footprint: two 1x19 female sock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"
- note added: "Wire colors are the breadboard jumpers in the owner photos (2026-09-24), not a harness specification. Inland e-paper driver board, write-only (GxEPD2_213_B74); no MISO. J2 pins follow the board header, pin 1 = SDI (top). Board switches P1 (3 / 0.47) and P2 (5VIN / 3.3VIN). Set P2 to 3.3VIN: J2 VCC is the DevKit 3.3 V rail (J19). Working unit: P1 on 3, P2 on 3.3VIN (photo, 2026-09-28)."
- note removed: "SCHEMATIC REVIEW / RELEASE HOLDS 1. U1 uses A1-A19 / J1-J19 from SigilBackMarked.png (BACK view); never exchange row identities. 2. U1 footprint (Sigil.pretty): 2.54 mm pitch, rows 22.86 mm (0.9 in) apart from the breadboard fit (Inland publishes 25.4 mm), 55.0 x 27.5 mm outline. Caliper-check and test-fit before ordering. 3. Future footprint: two 1x19 female sockets, unmistakable A1/J1 marks; ve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"
- note removed: "Wire colors are the breadboard jumpers in the owner photos (2026-09-24), not a harness specification. Inland e-paper driver board, write-only (GxEPD2_213_B74); no MISO. J2 pins follow the board header, pin 1 = SDI (top). Board switches P1 (3 / 0.47) and P2 (5VIN / 3.3VIN): positions not recorded; with the 3.3 V supply, check P2."
