File: KiCad/PCB/Sigilv1/Sigil_OLED.kicad_sch (KiCad schematic)
At the start: 13 parts, among them J2 INLAND 1.3" OLED HEADER (7-PI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, J3 BUZZER 2-PIN HEADER, J5 STATUS RING CABLE (JST-XH 3), SW1 UP (GPIO25, J11), SW2 DOWN (GPIO27, J9), SW3 LEFT (GPIO19, A12), SW4 RIGHT (GPIO21, A14), SW5 SELECT (GPIO32, J13), U1 REMOVABLE ESP32 DEVKIT / 2 x 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, U2 74AHCT1G125

Commit message: PCB Work
Parts:
- added C4: 100nF, Capacitor_THT:C_Disc_D5.0mm_W2.5mm_P5.00mm, symbol Sigil:Capacitor
- added J6: FRONT LIGHT CABLE (JST-XH 3), Connector_JST:JST_XH_B3B-XH-A_1x03_P2.50mm_Vertical, symbol Sigil:Front_Cable_JST_XH_3
- added R2: 330R, Resistor_THT:R_Axial_DIN0207_L6.3mm_D2.5mm_P7.62mm_Horizontal, symbol Sigil:Resistor_Series
- added U3: 74AHCT1G125, Package_TO_SOT_SMD:SOT-23-5, symbol Sigil:74AHCT1G125
Connections:
- net +5V: now also C4.1, J6.1 (+5V), U3.5 (VCC)
- net GND: now also C4.2, J6.3 (GND), U3.1 (OE#), U3.3 (GND)
- net FRONT_DIN: now reaches U1.J5 (GPIO13)
- net FRONT_DIN: now also U3.2 (A)
- new net FRONT_DIN_5V: R2.1, U3.4 (Y)
- new net FRONT_DIN_R: J6.2 (DIN), R2.2
- no-connect marks 20 -> 19
Other:
- note added: "FRONT LIGHT (SPARE OUTPUT)"
- note added: "J6: spare front light output, e.g. 6-8 SK6812 RGBW pixels on the case front lip facing the seated player. Own data line: GPIO13 -> U3 (74AHCT1G125, C4) -> R2 (330 ohm) -> DIN; pinout as J5. Shares USB 5V with the ring: firmware must cap both (7 + 8 pixels at 48/255 is about 225 mA). Fitted; unused until a strip is added."
- note added: "SCHEMATIC REVIEW / RELEASE HOLDS 1. U1 uses A1-A19 / J1-J19 from SigilBackMarked.png (BACK view); never exchange row identities. 2. U1 footprint (Sigil.pretty): 2.54 mm pitch, rows 22.86 mm (0.9 in) apart from the breadboard fit (Inland publishes 25.4 mm), 53.9 x 27.5 mm outline (length from the breadboard fit). Caliper-check and test-fit before ordering. 3. Future footprint: two 1x19 female sock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"
- note removed: "SCHEMATIC REVIEW / RELEASE HOLDS 1. U1 uses A1-A19 / J1-J19 from SigilBackMarked.png (BACK view); never exchange row identities. 2. U1 footprint (Sigil.pretty): 2.54 mm pitch, rows 22.86 mm (0.9 in) apart from the breadboard fit (Inland publishes 25.4 mm), 55.0 x 27.5 mm outline. Caliper-check and test-fit before ordering. 3. Future footprint: two 1x19 female sockets, unmistakable A1/J1 marks; ve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"
